Commit message: renamed to schunk_config

File: schunk_config/lwa/urdf/lwa.urdf.xacro (robot description, xacro)
@@ -4,14 +4,12 @@
        xmlns:interface="http://playerstage.sourceforge.net/gazebo/xmlschema/#interface"
        xmlns:xacro="http://playerstage.sourceforge.net/gazebo/xmlschema/#interface"
-       name="lwa_sdh" >
+       name="lwa" >
   <!-- common stuff -->
   <include filename="$(find cob_description)/urdf/common.xacro" />
   <include filename="$(find cob_description)/urdf/materials.urdf.xacro" />
   <!-- calibration -->
-  <include filename="$(find schunk_robots)/lwa_sdh/calibration/calibration.urdf.xacro" />
+  <include filename="$(find schunk_config)/lwa/calibration/calibration.urdf.xacro" />
   <!-- schunk lwa -->
   <include filename="$(find schunk_description)/urdf/lwa/lwa.urdf.xacro" />
-  <!-- schunk sdh -->
-  <include filename="$(find schunk_description)/urdf/sdh/sdh.urdf.xacro" />
   <!-- foot for arm -->
 	<link name="base_link">
@@ -35,11 +33,7 @@
 		</collision>
 	</link>
-  <!-- lwa -->
+  <!-- arm -->
   <xacro:schunk_lwa name="arm" parent="base_link">
     <origin xyz="0 0 0.5" rpy="3.1415926 0 0" />
   </xacro:schunk_lwa>
-  <!-- sdh -->
-  <xacro:schunk_sdh name="sdh" parent="arm_7_link">
-    <origin xyz="0 0 0" rpy="0 3.1415926 0" />
-  </xacro:schunk_sdh>
 </robot>

File: schunk_config/lwa_sdh/urdf/lwa_sdh.urdf.xacro (robot description, xacro)
@@ -4,12 +4,14 @@
        xmlns:interface="http://playerstage.sourceforge.net/gazebo/xmlschema/#interface"
        xmlns:xacro="http://playerstage.sourceforge.net/gazebo/xmlschema/#interface"
-       name="lwa" >
+       name="lwa_sdh" >
   <!-- common stuff -->
   <include filename="$(find cob_description)/urdf/common.xacro" />
   <include filename="$(find cob_description)/urdf/materials.urdf.xacro" />
   <!-- calibration -->
-  <include filename="$(find schunk_robots)/lwa/calibration/calibration.urdf.xacro" />
+  <include filename="$(find schunk_config)/lwa_sdh/calibration/calibration.urdf.xacro" />
   <!-- schunk lwa -->
   <include filename="$(find schunk_description)/urdf/lwa/lwa.urdf.xacro" />
+  <!-- schunk sdh -->
+  <include filename="$(find schunk_description)/urdf/sdh/sdh.urdf.xacro" />
   <!-- foot for arm -->
 	<link name="base_link">
@@ -33,7 +35,11 @@
 		</collision>
 	</link>
-  <!-- arm -->
+  <!-- lwa -->
   <xacro:schunk_lwa name="arm" parent="base_link">
     <origin xyz="0 0 0.5" rpy="3.1415926 0 0" />
   </xacro:schunk_lwa>
+  <!-- sdh -->
+  <xacro:schunk_sdh name="sdh" parent="arm_7_link">
+    <origin xyz="0 0 0" rpy="0 3.1415926 0" />
+  </xacro:schunk_sdh>
 </robot>
