Commit message: New mesh files for powerball

File: schunk_hardware_config/powerball/urdf/powerball.urdf.xacro (robot description, xacro)
@@ -36,5 +36,5 @@
   <!-- arm -->
   <xacro:schunk_powerball name="arm" parent="base_link">
-    <origin xyz="0 0 0.5" rpy="3.1415926 0 0" />
+    <origin xyz="0 0 0.54" rpy="0 0 0" />
   </xacro:schunk_powerball>
 </robot>

Commit message: Redefine powerball offset

File: schunk_hardware_config/powerball/urdf/powerball.urdf.xacro (robot description, xacro)
@@ -36,5 +36,5 @@
   <!-- arm -->
   <xacro:schunk_powerball name="arm" parent="base_link">
-    <origin xyz="0 0 0.54" rpy="0 0 0" />
+    <origin xyz="0 0 0.58" rpy="0 0 0" />
   </xacro:schunk_powerball>
 </robot>

Commit message: powerball

File: schunk_hardware_config/powerball/urdf/powerball.urdf.xacro (robot description, xacro)
@@ -36,5 +36,5 @@
   <!-- arm -->
   <xacro:schunk_powerball name="arm" parent="base_link">
-    <origin xyz="0 0 0.58" rpy="0 0 0" />
+    <origin xyz="0 0 0.5" rpy="${M_PI} 0 0" />
   </xacro:schunk_powerball>
 </robot>

Commit message: fix powerball urdf

File: schunk_hardware_config/powerball/urdf/powerball.urdf.xacro (robot description, xacro)
@@ -36,5 +36,5 @@
   <!-- arm -->
   <xacro:schunk_powerball name="arm" parent="base_link">
-    <origin xyz="0 0 0.5" rpy="${M_PI} 0 0" />
+    <origin xyz="0 0 0.58" rpy="0 0 0" />
   </xacro:schunk_powerball>
 </robot>

Commit message: Adjusted to joint for the new arm_0_link

File: schunk_hardware_config/powerball/urdf/powerball.urdf.xacro (robot description, xacro)
@@ -36,5 +36,5 @@
   <!-- arm -->
   <xacro:schunk_powerball name="arm" parent="base_link">
-    <origin xyz="0 0 0.58" rpy="0 0 0" />
+    <origin xyz="0 0 0.5" rpy="0 0 0" />
   </xacro:schunk_powerball>
 </robot>
