Commit message: Update sdh.urdf.xacro

File: schunk_hardware_config/sdh/urdf/sdh.urdf.xacro (robot description, xacro)
@@ -14,5 +14,5 @@
 	<link name="base_link">
 		<inertial>
-		   <origin xyz="0 0 -10" rpy="0 0 0"/>
+		   <origin xyz="0 0 -100" rpy="0 0 0"/>
 		   <mass value="1000.0"/>
 		   <inertia ixx="100.0"  ixy="0"  ixz="0" iyy="100.0" iyz="0" izz="100.0" />
