Commit message: Created lwa4d model

File: schunk_hardware_config/lwa4d/urdf/lwa4d.urdf.xacro (robot description, xacro)
@@ -36,5 +36,5 @@
   <!-- arm -->
   <xacro:schunk_lwa4d name="arm" parent="base_link">
-    <origin xyz="0 0 0.5" rpy="0 0 0" />
+    <origin xyz="0 0 0.5" rpy="0 0 -3.14159" />
   </xacro:schunk_lwa4d>
 </robot>

Commit message: Reset old version

File: schunk_hardware_config/lwa4d/urdf/lwa4d.urdf.xacro (robot description, xacro)
@@ -36,5 +36,5 @@
   <!-- arm -->
   <xacro:schunk_lwa4d name="arm" parent="base_link">
-    <origin xyz="0 0 0.5" rpy="0 0 -3.14159" />
+    <origin xyz="0 0 0.5" rpy="0 0 0" />
   </xacro:schunk_lwa4d>
 </robot>
