Commit message: Renamed the colors

File: schunk_hardware_config/lwa/urdf/lwa.urdf.xacro (robot description, xacro)
@@ -7,5 +7,5 @@
   <!-- common stuff -->
   <include filename="$(find cob_description)/urdf/common.xacro" />
-  <include filename="$(find cob_description)/urdf/materials.urdf.xacro" />
+  <include filename="$(find schunk_description)/urdf/materials.urdf.xacro" />
   <include filename="$(find cob_description)/gazebo/gazebo.urdf.xacro" />
   <!-- calibration -->
@@ -25,5 +25,5 @@
 			  <cylinder radius="0.1" length="0.5"/>
 		   </geometry>
-		   <material name="Grey" />
+		   <material name="IPA/DarkGrey" />
 		</visual>
 		<collision>

File: schunk_hardware_config/lwa_sdh/urdf/lwa_sdh.urdf.xacro (robot description, xacro)
@@ -7,5 +7,5 @@
   <!-- common stuff -->
   <include filename="$(find cob_description)/urdf/common.xacro" />
-  <include filename="$(find cob_description)/urdf/materials.urdf.xacro" />
+  <include filename="$(find schunk_description)/urdf/materials.urdf.xacro" />
   <include filename="$(find cob_description)/gazebo/gazebo.urdf.xacro" />
   <!-- calibration -->
@@ -27,5 +27,5 @@
 			  <cylinder radius="0.1" length="0.5"/>
 		   </geometry>
-		   <material name="Grey" />
+		   <material name="IPA/DarkGrey" />
 		</visual>
 		<collision>

File: schunk_hardware_config/powerball/urdf/powerball.urdf.xacro (robot description, xacro)
@@ -7,5 +7,5 @@
   <!-- common stuff -->
   <include filename="$(find cob_description)/urdf/common.xacro" />
-  <include filename="$(find cob_description)/urdf/materials.urdf.xacro" />
+  <include filename="$(find schunk_description)/urdf/materials.urdf.xacro" />
   <include filename="$(find cob_description)/gazebo/gazebo.urdf.xacro" />
   <!-- calibration -->
@@ -25,5 +25,5 @@
 			  <cylinder radius="0.1" length="0.5"/>
 		   </geometry>
-		   <material name="Grey" />
+		   <material name="IPA/DarkGrey" />
 		</visual>
 		<collision>

File: schunk_hardware_config/sdh/urdf/sdh.urdf.xacro (robot description, xacro)
@@ -7,5 +7,5 @@
   <!-- common stuff -->
   <include filename="$(find cob_description)/urdf/common.xacro" />
-  <include filename="$(find cob_description)/urdf/materials.urdf.xacro" />
+  <include filename="$(find schunk_description)/urdf/materials.urdf.xacro" />
   <include filename="$(find cob_description)/gazebo/gazebo.urdf.xacro" />
   <!-- schunk sdh -->
@@ -23,5 +23,5 @@
 			  <cylinder radius="0.1" length="0.5"/>
 		   </geometry>
-		   <material name="Grey" />
+		   <material name="IPA/DarkGrey" />
 		</visual>
 		<collision>

Commit message: rename color from IPA to Schunk

File: schunk_hardware_config/lwa/urdf/lwa.urdf.xacro (robot description, xacro)
@@ -25,5 +25,5 @@
 			  <cylinder radius="0.1" length="0.5"/>
 		   </geometry>
-		   <material name="IPA/DarkGrey" />
+		   <material name="Schunk/DarkGrey" />
 		</visual>
 		<collision>

File: schunk_hardware_config/lwa_sdh/urdf/lwa_sdh.urdf.xacro (robot description, xacro)
@@ -27,5 +27,5 @@
 			  <cylinder radius="0.1" length="0.5"/>
 		   </geometry>
-		   <material name="IPA/DarkGrey" />
+		   <material name="Schunk/DarkGrey" />
 		</visual>
 		<collision>

File: schunk_hardware_config/powerball/urdf/powerball.urdf.xacro (robot description, xacro)
@@ -25,5 +25,5 @@
 			  <cylinder radius="0.1" length="0.5"/>
 		   </geometry>
-		   <material name="IPA/DarkGrey" />
+		   <material name="Schunk/DarkGrey" />
 		</visual>
 		<collision>

File: schunk_hardware_config/sdh/urdf/sdh.urdf.xacro (robot description, xacro)
@@ -23,5 +23,5 @@
 			  <cylinder radius="0.1" length="0.5"/>
 		   </geometry>
-		   <material name="IPA/DarkGrey" />
+		   <material name="Schunk/DarkGrey" />
 		</visual>
 		<collision>

Commit message: Hydro migration

File: schunk_hardware_config/lwa/urdf/lwa.urdf.xacro (robot description, xacro)
@@ -1,16 +1,13 @@
 <?xml version="1.0"?>
-<robot xmlns:sensor="http://playerstage.sourceforge.net/gazebo/xmlschema/#sensor"
-       xmlns:controller="http://playerstage.sourceforge.net/gazebo/xmlschema/#controller"
-       xmlns:interface="http://playerstage.sourceforge.net/gazebo/xmlschema/#interface"
-       xmlns:xacro="http://playerstage.sourceforge.net/gazebo/xmlschema/#interface"
+<robot xmlns:xacro="http://playerstage.sourceforge.net/gazebo/xmlschema/#interface"
        name="lwa" >
   <!-- common stuff -->
-  <include filename="$(find cob_description)/urdf/common.xacro" />
-  <include filename="$(find schunk_description)/urdf/materials.urdf.xacro" />
-  <include filename="$(find cob_description)/gazebo/gazebo.urdf.xacro" />
+  <xacro:include filename="$(find cob_description)/urdf/common.xacro" />
+  <xacro:include filename="$(find schunk_description)/urdf/materials.urdf.xacro" />
+  <xacro:include filename="$(find cob_description)/gazebo/gazebo.urdf.xacro" />
   <!-- calibration -->
-  <include filename="$(find schunk_hardware_config)/lwa/calibration/calibration.urdf.xacro" />
+  <xacro:include filename="$(find schunk_hardware_config)/lwa/calibration/calibration.urdf.xacro" />
   <!-- schunk lwa -->
-  <include filename="$(find schunk_description)/urdf/lwa/lwa.urdf.xacro" />
+  <xacro:include filename="$(find schunk_description)/urdf/lwa/lwa.urdf.xacro" />
   <!-- foot for arm -->
 	<link name="base_link">

File: schunk_hardware_config/lwa4d/urdf/lwa4d.urdf.xacro (robot description, xacro)
@@ -1,16 +1,13 @@
 <?xml version="1.0"?>
-<robot xmlns:sensor="http://playerstage.sourceforge.net/gazebo/xmlschema/#sensor"
-       xmlns:controller="http://playerstage.sourceforge.net/gazebo/xmlschema/#controller"
-       xmlns:interface="http://playerstage.sourceforge.net/gazebo/xmlschema/#interface"
-       xmlns:xacro="http://playerstage.sourceforge.net/gazebo/xmlschema/#interface"
-       name="lwa4d" >
+<robot xmlns:xacro="http://www.ros.org/wiki/xacro"
+			 name="lwa4d" >
   <!-- common stuff -->
-  <include filename="$(find cob_description)/urdf/common.xacro" />
-  <include filename="$(find schunk_description)/urdf/materials.urdf.xacro" />
-  <include filename="$(find cob_description)/gazebo/gazebo.urdf.xacro" />
+  <xacro:include filename="$(find cob_description)/urdf/common.xacro" />
+  <xacro:include filename="$(find schunk_description)/urdf/materials.urdf.xacro" />
+  <xacro:include filename="$(find cob_description)/gazebo/gazebo.urdf.xacro" />
   <!-- calibration -->
-  <include filename="$(find schunk_hardware_config)/lwa4d/calibration/calibration.urdf.xacro" />
+  <xacro:include filename="$(find schunk_hardware_config)/lwa/calibration/calibration.urdf.xacro" />
   <!-- schunk lwa4d -->
-  <include filename="$(find schunk_description)/urdf/lwa4d/lwa4d.urdf.xacro" />
+  <xacro:include filename="$(find schunk_description)/urdf/lwa/lwa.urdf.xacro" />
   <!-- foot for arm -->
 	<link name="base_link">
@@ -35,6 +32,6 @@
 	</link>
   <!-- arm -->
-  <xacro:schunk_lwa4d name="arm" parent="base_link">
-    <origin xyz="0 0 0.5" rpy="0 0 0" />
-  </xacro:schunk_lwa4d>
+  <xacro:schunk_lwa name="arm" parent="base_link">
+    <origin xyz="0 0 0.5" rpy="0 3.14159 0" />
+  </xacro:schunk_lwa>
 </robot>

File: schunk_hardware_config/lwa4p/urdf/lwa4p.urdf.xacro (robot description, xacro)
@@ -1,16 +1,13 @@
 <?xml version="1.0"?>
-<robot xmlns:sensor="http://playerstage.sourceforge.net/gazebo/xmlschema/#sensor"
-       xmlns:controller="http://playerstage.sourceforge.net/gazebo/xmlschema/#controller"
-       xmlns:interface="http://playerstage.sourceforge.net/gazebo/xmlschema/#interface"
-       xmlns:xacro="http://playerstage.sourceforge.net/gazebo/xmlschema/#interface"
+<robot xmlns:xacro="http://playerstage.sourceforge.net/gazebo/xmlschema/#interface"
        name="lwa4p" >
   <!-- common stuff -->
-  <include filename="$(find cob_description)/urdf/common.xacro" />
-  <include filename="$(find schunk_description)/urdf/materials.urdf.xacro" />
-  <include filename="$(find cob_description)/gazebo/gazebo.urdf.xacro" />
+  <xacro:include filename="$(find cob_description)/urdf/common.xacro" />
+  <xacro:include filename="$(find schunk_description)/urdf/materials.urdf.xacro" />
+  <xacro:include filename="$(find cob_description)/gazebo/gazebo.urdf.xacro" />
   <!-- calibration -->
-  <include filename="$(find schunk_hardware_config)/lwa4p/calibration/calibration.urdf.xacro" />
+  <xacro:include filename="$(find schunk_hardware_config)/lwa4p/calibration/calibration.urdf.xacro" />
   <!-- schunk lwa4p -->
-  <include filename="$(find schunk_description)/urdf/lwa4p/lwa4p.urdf.xacro" />
+  <xacro:include filename="$(find schunk_description)/urdf/lwa4p/lwa4p.urdf.xacro" />
   <!-- foot for arm -->
 	<link name="base_link">

File: schunk_hardware_config/sdh/urdf/sdh.urdf.xacro (robot description, xacro)
@@ -1,14 +1,11 @@
 <?xml version="1.0"?>
-<robot xmlns:sensor="http://playerstage.sourceforge.net/gazebo/xmlschema/#sensor"
-       xmlns:controller="http://playerstage.sourceforge.net/gazebo/xmlschema/#controller"
-       xmlns:interface="http://playerstage.sourceforge.net/gazebo/xmlschema/#interface"
-       xmlns:xacro="http://playerstage.sourceforge.net/gazebo/xmlschema/#interface"
+<robot xmlns:xacro="http://playerstage.sourceforge.net/gazebo/xmlschema/#interface"
        name="sdh" >
   <!-- common stuff -->
-  <include filename="$(find cob_description)/urdf/common.xacro" />
-  <include filename="$(find schunk_description)/urdf/materials.urdf.xacro" />
-  <include filename="$(find cob_description)/gazebo/gazebo.urdf.xacro" />
+  <xacro:include filename="$(find cob_description)/urdf/common.xacro" />
+  <xacro:include filename="$(find schunk_description)/urdf/materials.urdf.xacro" />
+  <xacro:include filename="$(find cob_description)/gazebo/gazebo.urdf.xacro" />
   <!-- schunk sdh -->
-  <include filename="$(find schunk_description)/urdf/sdh/sdh.urdf.xacro" />
+  <xacro:include filename="$(find schunk_description)/urdf/sdh/sdh.urdf.xacro" />
   <!-- foot for arm -->
 	<link name="base_link">
