Commit message: fixes for example package

File: schunk_lwa4p/urdf/lwa4p.urdf.xacro (robot description, xacro)
@@ -14,24 +14,24 @@
   <include filename="$(find schunk_description)/urdf/lwa4p/lwa4p.urdf.xacro" />
   <!-- foot for arm -->
-	<link name="base_link">
-		<inertial>
-		   <origin xyz="0 0 -10" rpy="0 0 0"/>
-		   <mass value="1000.0"/>
-		   <inertia ixx="100.0"  ixy="0"  ixz="0" iyy="100.0" iyz="0" izz="100.0" />
-		</inertial>
-		<visual>
-		   <origin xyz="0 0 0.25" rpy="0 0 0" />
-		   <geometry>
-			  <cylinder radius="0.1" length="0.5"/>
-		   </geometry>
-		   <material name="Schunk/DarkGrey" />
-		</visual>
-		<collision>
-		   <origin xyz="0 0 0.25" rpy="0 0 0" />
-		   <geometry>
-			  <cylinder radius="0.1" length="0.5"/>
-		   </geometry>
-		</collision>
-	</link>
+  <link name="base_link">
+    <inertial>
+      <origin xyz="0 0 -10" rpy="0 0 0"/>
+      <mass value="1000.0"/>
+      <inertia ixx="100.0"  ixy="0"  ixz="0" iyy="100.0" iyz="0" izz="100.0" />
+    </inertial>
+    <visual>
+      <origin xyz="0 0 0.25" rpy="0 0 0" />
+      <geometry>
+         <cylinder radius="0.1" length="0.5"/>
+      </geometry>
+      <material name="Schunk/DarkGrey" />
+    </visual>
+    <collision>
+      <origin xyz="0 0 0.25" rpy="0 0 0" />
+      <geometry>
+        <cylinder radius="0.1" length="0.5"/>
+      </geometry>
+    </collision>
+  </link>
   <!-- arm -->
   <xacro:schunk_lwa4p name="arm" parent="base_link">
