Commit message: use inertias from CAD - first version

File: schunk_lwa4p_extended/urdf/common.xacro (robot description, xacro)
@@ -8,8 +8,8 @@
   <property name="cal_caster_br" value="0.0" />
   <!-- see https://secure.wikimedia.org/wikipedia/en/wiki/List_of_moment_of_inertia_tensors -->
-  <xacro:macro name="sphere_inertial" params="radius mass">
+  <xacro:macro name="sphere_inertial" params="radius mass *origin">
     <inertial>
       <mass value="${mass}" />
-      <origin xyz="0 0 0" />
+      <insert_block name="origin" />
       <inertia ixx="${0.4 * mass * radius * radius}" ixy="0.0" ixz="0.0"
         iyy="${0.4 * mass * radius * radius}" iyz="0.0"
@@ -17,8 +17,8 @@
     </inertial>
   </xacro:macro>
-  <xacro:macro name="cylinder_inertial" params="radius length mass">
+  <xacro:macro name="cylinder_inertial" params="radius length mass *origin">
     <inertial>
       <mass value="${mass}" />
-      <origin xyz="0 0 0" />
+      <insert_block name="origin" />
       <inertia ixx="${0.0833333 * mass * (3 * radius * radius + length * length)}" ixy="0.0" ixz="0.0"
         iyy="${0.0833333 * mass * (3 * radius * radius + length * length)}" iyz="0.0"
@@ -26,8 +26,8 @@
     </inertial>
   </xacro:macro>
-  <xacro:macro name="box_inertial" params="x y z mass">
+  <xacro:macro name="box_inertial" params="x y z mass *origin">
     <inertial>
       <mass value="${mass}" />
-      <origin xyz="0 0 0" />
+      <insert_block name="origin" />
       <inertia ixx="${0.0833333 * mass * (y*y + z*z)}" ixy="0.0" ixz="0.0"
         iyy="${0.0833333 * mass * (x*x + z*z)}" iyz="0.0"

File: schunk_lwa4p_extended/urdf/lwa4p_extended.gazebo.xacro (robot description, xacro)
@@ -2,5 +2,5 @@
 <robot xmlns:xacro="http://www.ros.org/wiki/xacro">
   <xacro:macro name="schunk_lwa4p_extended_gazebo" params="name">
-    <gazebo reference="${name}_0_link">
+    <gazebo reference="${name}_base_link">
       <material value="Schunk/LightGrey" />
       <turnGravityOff>false</turnGravityOff>

File: schunk_lwa4p_extended/urdf/lwa4p_extended.urdf.xacro (robot description, xacro)
@@ -11,9 +11,7 @@
     </joint>
     <link name="${name}_base_link">
-      <inertial>
-        <origin xyz="0 0 0" rpy="0 0 0"/>
-        <mass value="0.1"/>
-        <inertia ixx="0.01" ixy="0" ixz="0" iyy="0.01" iyz="0" izz="0.01" />
-      </inertial>
+      <xacro:cylinder_inertial radius="0.056" length="0.134" mass="2.0">
+        <origin xyz="0 0 ${0.134/2}" rpy="0 0 0" />
+      </xacro:cylinder_inertial>
       <visual>
         <origin xyz="0 0 0" rpy="0 0 0" />
@@ -41,9 +39,7 @@
     </joint>
     <link name="${name}_1_link">
-      <inertial>
-        <origin xyz="0 0 0" rpy="0 0 0"/>
-        <mass value="0.1"/>
-        <inertia ixx="0.01" ixy="0" ixz="0" iyy="0.01" iyz="0" izz="0.01" />
-      </inertial>
+      <xacro:box_inertial x="0.01" y="0.01" z="0.01" mass="0.1">
+        <origin xyz="0 0 0" rpy="0 0 0" />
+      </xacro:box_inertial>
       <visual>
         <origin xyz="0 0 0" rpy="0 0 0" />
@@ -74,7 +70,7 @@
     <link name="${name}_2_link">
       <inertial>
-        <origin xyz="0 0 0" rpy="0 0 0"/>
-        <mass value="0.1"/>
-        <inertia ixx="0.01" ixy="0" ixz="0" iyy="0.01" iyz="0" izz="0.01" />
+        <origin xyz="0 0.018 0.018" rpy="0 0 0"/>
+        <mass value="3.9"/>
+        <inertia ixx="0.009780" ixy="0.0" ixz="0.0" iyy="0.013300" iyz="0.0" izz="0.009780" />
       </inertial>
       <visual>
@@ -104,7 +100,7 @@
     <link name="${name}_3_link">
       <inertial>
-        <origin xyz="0 0 0" rpy="0 0 0"/>
-        <mass value="0.1"/>
-        <inertia ixx="0.01" ixy="0" ixz="0" iyy="0.01" iyz="0" izz="0.01" />
+        <origin xyz="0.0 0.06247 0.23425" rpy="0 0 0"/>
+        <mass value="1.94533"/>
+        <inertia ixx="0.0344" ixy="0.0" ixz="0.0077" iyy="0.0362" iyz="0.0" izz="0.0052" />
       </inertial>
       <inertial>
@@ -139,7 +135,7 @@
     <link name="${name}_4_link">
       <inertial>
-        <origin xyz="0 0 0" rpy="0 0 0"/>
-        <mass value="0.1"/>
-        <inertia ixx="0.01" ixy="0" ixz="0" iyy="0.01" iyz="0" izz="0.01" />
+        <origin xyz="0 0.018 -0.018" rpy="0 0 0"/>
+        <mass value="3.9"/>
+        <inertia ixx="0.009780" ixy="0.0" ixz="0.0" iyy="0.013300" iyz="0.0" izz="0.009780" />
       </inertial>
       <visual>
@@ -169,7 +165,7 @@
     <link name="${name}_5_link">
       <inertial>
-        <origin xyz="0 0 0" rpy="0 0 0"/>
-        <mass value="0.1"/>
-        <inertia ixx="0.01" ixy="0" ixz="0" iyy="0.01" iyz="0" izz="0.01" />
+        <origin xyz="0.0 0.04175 0.17026" rpy="0 0 0"/>
+        <mass value="1.3297"/>
+        <inertia ixx="0.01" ixy="0.0" ixz="-0.0031" iyy="0.0111" iyz="0.0" izz="0.0031" />
       </inertial>
       <visual>
@@ -199,7 +195,7 @@
     <link name="${name}_6_link">
       <inertial>
-        <origin xyz="0 0 0" rpy="0 0 0"/>
-        <mass value="0.1"/>
-        <inertia ixx="0.01" ixy="0" ixz="0" iyy="0.01" iyz="0" izz="0.01" />
+        <origin xyz="0 0.012 -0.012" rpy="0 0 0"/>
+        <mass value="1.9"/>
+        <inertia ixx="0.002750" ixy="0.0" ixz="0.0" iyy="0.004002" iyz="0.0" izz="0.002830" />
       </inertial>
       <visual>
@@ -233,19 +229,22 @@
         <inertia ixx="0.01" ixy="0" ixz="0" iyy="0.01" iyz="0" izz="0.01" />
       </inertial>
-      <visual>
-        <origin xyz="0 0 0" rpy="0 0 0" />
-        <geometry>
-          <!--mesh filename="package://schunk_lwa4p_extended/meshes/arm_7_link.stl" /-->
-          <box size="0.05 0.05 0.05"/>
-        </geometry>
-      </visual>
-      <collision>
-        <origin xyz="0 0 0" rpy="0 0 0" />
-        <geometry>
-          <!--mesh filename="package://schunk_lwa4p_extended/meshes/arm_7_link.stl" /-->
-          <box size="0.05 0.05 0.05"/>
-        </geometry>
-      </collision>
-    </link>
+    </link>
+    <!--link name="${name}_7_link">
+      <xacro:box_inertial x="0.01" y="0.01" z="0.01" mass="0.1">
+        <origin xyz="0 0 0" rpy="0 0 0" />
+      </xacro:box_inertial>
+      <visual>
+        <origin xyz="0 0 0" rpy="0 0 0" />
+        <geometry>
+          <box size="0.01 0.01 0.01"/>
+        </geometry>
+      </visual>
+      <collision>
+        <origin xyz="0 0 0" rpy="0 0 0" />
+        <geometry>
+          <box size="0.01 0.01 0.01"/>
+        </geometry>
+      </collision>
+    </link-->
     <!-- extensions -->
     <xacro:schunk_lwa4p_extended_gazebo name="${name}" />

File: schunk_lwa4p_extended/urdf/robot_lwa4p_extended.urdf.xacro (robot description, xacro)
@@ -10,27 +10,8 @@
   <!-- schunk lwa4p_extended -->
   <xacro:include filename="$(find schunk_lwa4p_extended)/urdf/lwa4p_extended.urdf.xacro" />
-  <!-- foot for arm -->
-  <link name="base_link">
-    <inertial>
-      <origin xyz="0 0 -10" rpy="0 0 0"/>
-      <mass value="1000.0"/>
-      <inertia ixx="100.0"  ixy="0"  ixz="0" iyy="100.0" iyz="0" izz="100.0" />
-    </inertial>
-    <visual>
-      <origin xyz="0 0 0.25" rpy="0 0 0" />
-      <geometry>
-         <cylinder radius="0.1" length="0.5"/>
-      </geometry>
-      <material name="Schunk/DarkGrey" />
-    </visual>
-    <collision>
-      <origin xyz="0 0 0.25" rpy="0 0 0" />
-      <geometry>
-        <cylinder radius="0.1" length="0.5"/>
-      </geometry>
-    </collision>
-  </link>
+  <!-- Used for fixing robot to Gazebo 'base_link' -->
+  <link name="world"/>
   <!-- arm -->
-  <xacro:schunk_lwa4p_extended name="arm" parent="base_link"
+  <xacro:schunk_lwa4p_extended name="arm" parent="world"
             arm_1_ref="${arm_1_ref}"
             arm_2_ref="${arm_2_ref}"
@@ -40,5 +21,5 @@
             arm_6_ref="${arm_6_ref}"
             arm_7_ref="${arm_7_ref}">
-    <origin xyz="0 0 0.5" rpy="0 0 0" />
+    <origin xyz="0 0 0" rpy="0 0 0" />
   </xacro:schunk_lwa4p_extended>
 </robot>
