Commit message: be independend from schunk_modular_robotics and cob_common to be able to test inertia and controllers seperately

File: schunk_lwa4p_extended/urdf/lwa4p_extended.urdf.xacro (robot description, xacro)
@@ -1,44 +1,214 @@
 <?xml version="1.0"?>
-<robot xmlns:xacro="http://www.ros.org/wiki/xacro"
-       name="lwa4p_extended" >
-  <!-- common stuff -->
-  <xacro:include filename="$(find cob_description)/urdf/common.xacro" />
-  <xacro:include filename="$(find schunk_description)/urdf/materials.urdf.xacro" />
-  <xacro:include filename="$(find cob_description)/gazebo/gazebo.urdf.xacro" />
-  <!-- calibration -->
-  <xacro:include filename="$(find schunk_lwa4p_extended)/calibration/calibration.urdf.xacro" />
-  <!-- schunk lwa4p_extended -->
-  <xacro:include filename="$(find schunk_description)/urdf/lwa4p_extended/lwa4p_extended.urdf.xacro" />
-  <!-- foot for arm -->
-  <link name="base_link">
-    <inertial>
-      <origin xyz="0 0 -10" rpy="0 0 0"/>
-      <mass value="1000.0"/>
-      <inertia ixx="100.0"  ixy="0"  ixz="0" iyy="100.0" iyz="0" izz="100.0" />
-    </inertial>
+<robot xmlns:xacro="http://www.ros.org/wiki/xacro">
+  <xacro:include filename="$(find schunk_lwa4p_extended)/urdf/lwa4p_extended.gazebo.xacro" />
+  <xacro:include filename="$(find schunk_lwa4p_extended)/urdf/lwa4p_extended.transmission.xacro" />
+  <xacro:macro name="schunk_lwa4p_extended" params="parent name *origin arm_1_ref arm_2_ref arm_3_ref arm_4_ref arm_5_ref arm_6_ref arm_7_ref">
+    <!-- joint between base_link and lwa4p_extended_connector_link -->
+    <joint name="${name}_base_joint" type="fixed">
+      <insert_block name="origin" />
+      <parent link="${parent}"/>
+      <child link="${name}_base_link"/>
+    </joint>
+    <link name="${name}_base_link">
+      <inertial>
+        <origin xyz="0 0 0" rpy="0 0 0"/>
+        <mass value="0.1"/>
+        <inertia ixx="0.01" ixy="0" ixz="0" iyy="0.01" iyz="0" izz="0.01" />
+      </inertial>
+    </link>
+    <!-- joint between arm_base_link and arm_1_link -->
+    <joint name="${name}_1_joint" type="revolute" >
+      <origin xyz="0 0 0" rpy="0 0 0" />
+      <parent link="${name}_base_link" />
+      <child link="${name}_1_link" />
+      <axis xyz="0 0 1"/>
+      <calibration rising="${arm_1_ref}"/>
+      <dynamics damping="10" />
+      <limit effort="370" velocity="2.0" lower="-6.2831853" upper="6.2831853"/>
+      <safety_controller k_position="20" k_velocity="50" soft_lower_limit="${-6.2831853 + 0.01}" soft_upper_limit="${6.2831853 - 0.01}" />
+    </joint>
+    <link name="${name}_1_link">
+      <inertial>
+        <origin xyz="0 0 0" rpy="0 0 0"/>
+        <mass value="0.1"/>
+        <inertia ixx="0.01" ixy="0" ixz="0" iyy="0.01" iyz="0" izz="0.01" />
+      </inertial>
+    </link>
+    <!-- joint between arm_1_link and arm_2_link -->
+    <joint name="${name}_2_joint" type="revolute">
+      <origin xyz="0 0 0.0915" rpy="1.5708 0 0"/>
+      <parent link="${name}_1_link"/>
+      <child link="${name}_2_link"/>
+      <axis xyz="0 0 1"/>
+      <calibration rising="${arm_2_ref}"/>
+      <dynamics damping="10" />
+      <limit effort="370" velocity="2.0" lower="-2.0943951" upper="2.0943951"/>
+      <safety_controller k_position="20" k_velocity="50" soft_lower_limit="${-2.0943 + 0.01}" soft_upper_limit="${2.0943 - 0.01}" />
+    </joint>
+    <link name="${name}_2_link">
+      <inertial>
+        <origin xyz="0 0 0" rpy="0 0 0"/>
+        <mass value="0.1"/>
+        <inertia ixx="0.01" ixy="0" ixz="0" iyy="0.01" iyz="0" izz="0.01" />
+      </inertial>
     <visual>
-      <origin xyz="0 0 0.25" rpy="0 0 0" />
-      <geometry>
-         <cylinder radius="0.1" length="0.5"/>
-      </geometry>
-      <material name="Schunk/DarkGrey" />
-    </visual>
-    <collision>
-      <origin xyz="0 0 0.25" rpy="0 0 0" />
-      <geometry>
-        <cylinder radius="0.1" length="0.5"/>
-      </geometry>
-    </collision>
-  </link>
-  <!-- arm -->
-  <xacro:schunk_lwa4p_extended name="arm" parent="base_link"
-            arm_1_ref="${arm_1_ref}"
-            arm_2_ref="${arm_2_ref}"
-            arm_3_ref="${arm_3_ref}"
-            arm_4_ref="${arm_4_ref}"
-            arm_5_ref="${arm_5_ref}"
-            arm_6_ref="${arm_6_ref}"
-            arm_7_ref="${arm_7_ref}">
-    <origin xyz="0 0 0.5" rpy="0 0 0" />
-  </xacro:schunk_lwa4p_extended>
+        <origin xyz="0 0 0" rpy="0 0 0" />
+        <geometry>
+          <mesh filename="package://schunk_lwa4p_extended/meshes/arm_1_link.dae" />
+        </geometry>
+      </visual>
+      <collision>
+        <origin xyz="0 0 0" rpy="0 0 0" />
+        <geometry>
+          <mesh filename="package://schunk_lwa4p_extended/meshes/arm_1_link.dae" />
+        </geometry>
+      </collision>
+    </link>
+    <!-- joint between arm_2_link and arm_3_link -->
+    <joint name="${name}_3_joint" type="revolute">
+      <origin xyz="0 0 0" rpy="-1.5708 0 0"/>
+      <parent link="${name}_2_link"/>
+      <child link="${name}_3_link"/>
+      <axis xyz="0 0 1"/>
+      <calibration rising="${arm_3_ref}"/>
+      <dynamics damping="5" />
+      <limit effort="176" velocity="2.0" lower="-6.2831853" upper="6.2831853"/>
+      <safety_controller k_position="20" k_velocity="25" soft_lower_limit="${-6.2831853 + 0.01}" soft_upper_limit="${6.2831853 - 0.01}" />
+    </joint>
+    <link name="${name}_3_link">
+      <inertial>
+        <origin xyz="0 0 0" rpy="0 0 0"/>
+        <mass value="0.1"/>
+        <inertia ixx="0.01" ixy="0" ixz="0" iyy="0.01" iyz="0" izz="0.01" />
+      </inertial>
+      <inertial>
+        <origin xyz="0 0 0" rpy="0 0 0"/>
+        <mass value="0.1"/>
+        <inertia ixx="0.01" ixy="0" ixz="0" iyy="0.01" iyz="0" izz="0.01" />
+      </inertial>
+    <visual>
+        <origin xyz="0 0 0" rpy="0 0 0" />
+        <geometry>
+          <mesh filename="package://schunk_lwa4p_extended/meshes/arm_2_link.dae" />
+        </geometry>
+      </visual>
+      <collision>
+        <origin xyz="0 0 0" rpy="0 0 0" />
+        <geometry>
+          <mesh filename="package://schunk_lwa4p_extended/meshes/arm_2_link.dae" />
+        </geometry>
+      </collision>
+    </link>
+    <!-- joint between arm_3_link and arm_4_link -->
+    <joint name="${name}_4_joint" type="revolute">
+      <origin xyz="0 0 0.45360" rpy="1.5708 0 0" />
+      <parent link="${name}_3_link"/>
+      <child link="${name}_4_link"/>
+      <axis xyz="0 0 1" />
+      <calibration rising="${arm_4_ref}"/>
+      <dynamics damping="5" />
+      <limit effort="176" velocity="2.0" lower="-2.0943951" upper="2.0943951"/>
+      <safety_controller k_position="20" k_velocity="25" soft_lower_limit="${-2.0943951 + 0.01}" soft_upper_limit="${2.0943951 - 0.01}" />
+    </joint>
+    <link name="${name}_4_link">
+      <inertial>
+        <origin xyz="0 0 0" rpy="0 0 0"/>
+        <mass value="0.1"/>
+        <inertia ixx="0.01" ixy="0" ixz="0" iyy="0.01" iyz="0" izz="0.01" />
+      </inertial>
+      <visual>
+        <origin xyz="0 0 0" rpy="0 0 0" />
+        <geometry>
+          <mesh filename="package://schunk_lwa4p_extended/meshes/arm_3_link.dae" />
+        </geometry>
+      </visual>
+      <collision>
+        <origin xyz="0 0 0" rpy="0 0 0" />
+        <geometry>
+          <mesh filename="package://schunk_lwa4p_extended/meshes/arm_3_link.dae" />
+        </geometry>
+      </collision>
+    </link>
+    <!-- joint between arm_4_link and arm_5_link -->
+    <joint name="${name}_5_joint" type="revolute">
+      <origin xyz="0 0 0" rpy="-1.5708 0 0" />
+      <parent link="${name}_4_link"/>
+      <child link="${name}_5_link"/>
+      <axis xyz="0 0 1" />
+      <calibration rising="${arm_5_ref}"/>
+      <dynamics damping="5" />
+      <limit effort="41.6" velocity="2.0" lower="-6.2831853" upper="6.2831853" />
+      <safety_controller k_position="20" k_velocity="25" soft_lower_limit="${-6.2831853 + 0.01}" soft_upper_limit="${6.2831853 - 0.01}" />
+    </joint>
+    <link name="${name}_5_link">
+      <inertial>
+        <origin xyz="0 0 0" rpy="0 0 0"/>
+        <mass value="0.1"/>
+        <inertia ixx="0.01" ixy="0" ixz="0" iyy="0.01" iyz="0" izz="0.01" />
+      </inertial>
+      <visual>
+        <origin xyz="0 0 0" rpy="0 0 0" />
+        <geometry>
+          <mesh filename="package://schunk_lwa4p_extended/meshes/arm_4_link.dae" />
+        </geometry>
+      </visual>
+      <collision>
+        <origin xyz="0 0 0" rpy="0 0 0" />
+        <geometry>
+          <mesh filename="package://schunk_lwa4p_extended/meshes/arm_4_link.dae" />
+        </geometry>
+      </collision>
+    </link>
+    <!-- joint between arm_5_link and arm_6_link -->
+    <joint name="${name}_6_joint" type="revolute">
+      <origin xyz="0 0 0.2986" rpy="1.5708 0 0" />
+      <parent link="${name}_5_link"/>
+      <child link="${name}_6_link"/>
+      <axis xyz="0 0 1" />
+      <calibration rising="${arm_6_ref}"/>
+      <dynamics damping="5" />
+      <limit effort="20.1" velocity="2.0" lower="-2.0943951" upper="2.0943951" />
+      <safety_controller k_position="20" k_velocity="25" soft_lower_limit="${-2.0943951 + 0.01}" soft_upper_limit="${2.0943951 - 0.01}" />
+    </joint>
+    <link name="${name}_6_link">
+      <inertial>
+        <origin xyz="0 0 0" rpy="0 0 0"/>
+        <mass value="0.1"/>
+        <inertia ixx="0.01" ixy="0" ixz="0" iyy="0.01" iyz="0" izz="0.01" />
+      </inertial>
+      <visual>
+        <origin xyz="0 0 0" rpy="0 0 0" />
+        <geometry>
+          <mesh filename="package://schunk_lwa4p_extended/meshes/arm_5_link.dae" />
+        </geometry>
+      </visual>
+      <collision>
+        <origin xyz="0 0 0" rpy="0 0 0" />
+        <geometry>
+          <mesh filename="package://schunk_lwa4p_extended/meshes/arm_5_link.dae" />
+        </geometry>
+      </collision>
+    </link>
+    <!-- joint between arm_6_link and arm_7_link -->
+    <joint name="${name}_7_joint" type="revolute">
+      <origin xyz="0 0 0" rpy="-1.5708 0 0" />
+      <parent link="${name}_6_link"/>
+      <child link="${name}_7_link"/>
+      <axis xyz="0 0 1" />
+      <calibration rising="${arm_7_ref}"/>
+      <dynamics damping="5" />
+      <limit effort="20.1" velocity="2.0" lower="-2.0943951" upper="2.0943951" />
+      <safety_controller k_position="20" k_velocity="25" soft_lower_limit="${-2.0943951 + 0.01}" soft_upper_limit="${2.0943951 - 0.01}" />
+    </joint>
+    <link name="${name}_7_link">
+      <inertial>
+        <origin xyz="0 0 0" rpy="0 0 0"/>
+        <mass value="0.1"/>
+        <inertia ixx="0.01" ixy="0" ixz="0" iyy="0.01" iyz="0" izz="0.01" />
+      </inertial>
+    </link>
+    <!-- extensions -->
+    <xacro:schunk_lwa4p_extended_gazebo name="${name}" />
+    <xacro:schunk_lwa4p_extended_transmission name="${name}" />
+  </xacro:macro>
 </robot>

Commit message: fixed mesh numbering + new mesh for prl100

File: schunk_lwa4p_extended/urdf/lwa4p_extended.urdf.xacro (robot description, xacro)
@@ -16,8 +16,20 @@
         <inertia ixx="0.01" ixy="0" ixz="0" iyy="0.01" iyz="0" izz="0.01" />
       </inertial>
+      <visual>
+        <origin xyz="0 0 0" rpy="0 0 0" />
+        <geometry>
+          <mesh filename="package://schunk_lwa4p_extended/meshes/arm_base_link.stl" />
+        </geometry>
+      </visual>
+      <collision>
+        <origin xyz="0 0 0" rpy="0 0 0" />
+        <geometry>
+          <mesh filename="package://schunk_lwa4p_extended/meshes/arm_base_link.stl" />
+        </geometry>
+      </collision>
     </link>
     <!-- joint between arm_base_link and arm_1_link -->
     <joint name="${name}_1_joint" type="revolute" >
-      <origin xyz="0 0 0" rpy="0 0 0" />
+      <origin xyz="0 0 ${0.134+0.005}" rpy="0 0 0" />
       <parent link="${name}_base_link" />
       <child link="${name}_1_link" />
@@ -34,4 +46,18 @@
         <inertia ixx="0.01" ixy="0" ixz="0" iyy="0.01" iyz="0" izz="0.01" />
       </inertial>
+      <visual>
+        <origin xyz="0 0 0" rpy="0 0 0" />
+        <geometry>
+          <!--mesh filename="package://schunk_lwa4p_extended/meshes/arm_1_link.stl" /-->
+          <box size="0.01 0.01 0.01"/>
+        </geometry>
+      </visual>
+      <collision>
+        <origin xyz="0 0 0" rpy="0 0 0" />
+        <geometry>
+          <!--mesh filename="package://schunk_lwa4p_extended/meshes/arm_1_link.stl" /-->
+          <box size="0.01 0.01 0.01"/>
+        </geometry>
+      </collision>
     </link>
     <!-- joint between arm_1_link and arm_2_link -->
@@ -52,14 +78,14 @@
         <inertia ixx="0.01" ixy="0" ixz="0" iyy="0.01" iyz="0" izz="0.01" />
       </inertial>
-    <visual>
-        <origin xyz="0 0 0" rpy="0 0 0" />
-        <geometry>
-          <mesh filename="package://schunk_lwa4p_extended/meshes/arm_1_link.dae" />
-        </geometry>
-      </visual>
-      <collision>
-        <origin xyz="0 0 0" rpy="0 0 0" />
-        <geometry>
-          <mesh filename="package://schunk_lwa4p_extended/meshes/arm_1_link.dae" />
+      <visual>
+        <origin xyz="0 0 0" rpy="0 0 0" />
+        <geometry>
+          <mesh filename="package://schunk_lwa4p_extended/meshes/arm_2_link.dae" />
+        </geometry>
+      </visual>
+      <collision>
+        <origin xyz="0 0 0" rpy="0 0 0" />
+        <geometry>
+          <mesh filename="package://schunk_lwa4p_extended/meshes/arm_2_link.dae" />
         </geometry>
       </collision>
@@ -90,11 +116,11 @@
         <origin xyz="0 0 0" rpy="0 0 0" />
         <geometry>
-          <mesh filename="package://schunk_lwa4p_extended/meshes/arm_2_link.dae" />
-        </geometry>
-      </visual>
-      <collision>
-        <origin xyz="0 0 0" rpy="0 0 0" />
-        <geometry>
-          <mesh filename="package://schunk_lwa4p_extended/meshes/arm_2_link.dae" />
+          <mesh filename="package://schunk_lwa4p_extended/meshes/arm_3_link.dae" />
+        </geometry>
+      </visual>
+      <collision>
+        <origin xyz="0 0 0" rpy="0 0 0" />
+        <geometry>
+          <mesh filename="package://schunk_lwa4p_extended/meshes/arm_3_link.dae" />
         </geometry>
       </collision>
@@ -120,11 +146,11 @@
         <origin xyz="0 0 0" rpy="0 0 0" />
         <geometry>
-          <mesh filename="package://schunk_lwa4p_extended/meshes/arm_3_link.dae" />
-        </geometry>
-      </visual>
-      <collision>
-        <origin xyz="0 0 0" rpy="0 0 0" />
-        <geometry>
-          <mesh filename="package://schunk_lwa4p_extended/meshes/arm_3_link.dae" />
+          <mesh filename="package://schunk_lwa4p_extended/meshes/arm_4_link.dae" />
+        </geometry>
+      </visual>
+      <collision>
+        <origin xyz="0 0 0" rpy="0 0 0" />
+        <geometry>
+          <mesh filename="package://schunk_lwa4p_extended/meshes/arm_4_link.dae" />
         </geometry>
       </collision>
@@ -150,11 +176,11 @@
         <origin xyz="0 0 0" rpy="0 0 0" />
         <geometry>
-          <mesh filename="package://schunk_lwa4p_extended/meshes/arm_4_link.dae" />
-        </geometry>
-      </visual>
-      <collision>
-        <origin xyz="0 0 0" rpy="0 0 0" />
-        <geometry>
-          <mesh filename="package://schunk_lwa4p_extended/meshes/arm_4_link.dae" />
+          <mesh filename="package://schunk_lwa4p_extended/meshes/arm_5_link.dae" />
+        </geometry>
+      </visual>
+      <collision>
+        <origin xyz="0 0 0" rpy="0 0 0" />
+        <geometry>
+          <mesh filename="package://schunk_lwa4p_extended/meshes/arm_5_link.dae" />
         </geometry>
       </collision>
@@ -180,11 +206,11 @@
         <origin xyz="0 0 0" rpy="0 0 0" />
         <geometry>
-          <mesh filename="package://schunk_lwa4p_extended/meshes/arm_5_link.dae" />
-        </geometry>
-      </visual>
-      <collision>
-        <origin xyz="0 0 0" rpy="0 0 0" />
-        <geometry>
-          <mesh filename="package://schunk_lwa4p_extended/meshes/arm_5_link.dae" />
+          <mesh filename="package://schunk_lwa4p_extended/meshes/arm_6_link.dae" />
+        </geometry>
+      </visual>
+      <collision>
+        <origin xyz="0 0 0" rpy="0 0 0" />
+        <geometry>
+          <mesh filename="package://schunk_lwa4p_extended/meshes/arm_6_link.dae" />
         </geometry>
       </collision>
@@ -207,4 +233,18 @@
         <inertia ixx="0.01" ixy="0" ixz="0" iyy="0.01" iyz="0" izz="0.01" />
       </inertial>
+      <visual>
+        <origin xyz="0 0 0" rpy="0 0 0" />
+        <geometry>
+          <!--mesh filename="package://schunk_lwa4p_extended/meshes/arm_7_link.stl" /-->
+          <box size="0.05 0.05 0.05"/>
+        </geometry>
+      </visual>
+      <collision>
+        <origin xyz="0 0 0" rpy="0 0 0" />
+        <geometry>
+          <!--mesh filename="package://schunk_lwa4p_extended/meshes/arm_7_link.stl" /-->
+          <box size="0.05 0.05 0.05"/>
+        </geometry>
+      </collision>
     </link>
     <!-- extensions -->

Commit message: update effort limits

File: schunk_lwa4p_extended/urdf/lwa4p_extended.urdf.xacro (robot description, xacro)
@@ -35,5 +35,5 @@
       <calibration rising="${arm_1_ref}"/>
       <dynamics damping="1" friction="0"/> <!-- default_damping = 0 [N], default_friction = 0 -->
-      <limit effort="370" velocity="2.0" lower="-6.2831853" upper="6.2831853"/>
+      <limit effort="81.5" velocity="0.42" lower="-6.2831853" upper="6.2831853"/>
       <safety_controller k_position="20" k_velocity="50" soft_lower_limit="${-6.2831853 + 0.01}" soft_upper_limit="${6.2831853 - 0.01}" />
     </joint>
@@ -65,5 +65,5 @@
       <calibration rising="${arm_2_ref}"/>
       <dynamics damping="1"/>
-      <limit effort="370" velocity="2.0" lower="-2.0943951" upper="2.0943951"/>
+      <limit effort="38" velocity="26.1" lower="-2.0943951" upper="2.0943951"/>
       <safety_controller k_position="20" k_velocity="50" soft_lower_limit="${-2.0943 + 0.01}" soft_upper_limit="${2.0943 - 0.01}" />
     </joint>
@@ -95,5 +95,5 @@
       <calibration rising="${arm_3_ref}"/>
       <dynamics damping="1" />
-      <limit effort="176" velocity="2.0" lower="-6.2831853" upper="6.2831853"/>
+      <limit effort="38" velocity="26.1" lower="-6.2831853" upper="6.2831853"/>
       <safety_controller k_position="20" k_velocity="25" soft_lower_limit="${-6.2831853 + 0.01}" soft_upper_limit="${6.2831853 - 0.01}" />
     </joint>
@@ -130,5 +130,5 @@
       <calibration rising="${arm_4_ref}"/>
       <dynamics damping="1"/>
-      <limit effort="176" velocity="2.0" lower="-2.0943951" upper="2.0943951"/>
+      <limit effort="38" velocity="26.1" lower="-2.0943951" upper="2.0943951"/>
       <safety_controller k_position="20" k_velocity="25" soft_lower_limit="${-2.0943951 + 0.01}" soft_upper_limit="${2.0943951 - 0.01}" />
     </joint>
@@ -160,5 +160,5 @@
       <calibration rising="${arm_5_ref}"/>
       <dynamics damping="1" />
-      <limit effort="41.6" velocity="2.0" lower="-6.2831853" upper="6.2831853" />
+      <limit effort="38" velocity="26.1" lower="-6.2831853" upper="6.2831853" />
       <safety_controller k_position="20" k_velocity="25" soft_lower_limit="${-6.2831853 + 0.01}" soft_upper_limit="${6.2831853 - 0.01}" />
     </joint>
@@ -190,5 +190,5 @@
       <calibration rising="${arm_6_ref}"/>
       <dynamics damping="1" />
-      <limit effort="20.1" velocity="2.0" lower="-2.0943951" upper="2.0943951" />
+      <limit effort="15" velocity="24.9" lower="-2.0943951" upper="2.0943951" />
       <safety_controller k_position="20" k_velocity="25" soft_lower_limit="${-2.0943951 + 0.01}" soft_upper_limit="${2.0943951 - 0.01}" />
     </joint>
@@ -220,5 +220,5 @@
       <calibration rising="${arm_7_ref}"/>
       <dynamics damping="1" />
-      <limit effort="20.1" velocity="2.0" lower="-2.0943951" upper="2.0943951" />
+      <limit effort="15" velocity="24.9" lower="-2.0943951" upper="2.0943951" />
       <safety_controller k_position="20" k_velocity="25" soft_lower_limit="${-2.0943951 + 0.01}" soft_upper_limit="${2.0943951 - 0.01}" />
     </joint>

Commit message: use values from CAD and datasheet

File: schunk_lwa4p_extended/urdf/lwa4p_extended.urdf.xacro (robot description, xacro)
@@ -52,5 +52,4 @@
         <origin xyz="0 0 0" rpy="0 0 0" />
         <geometry>
-          <!--mesh filename="package://schunk_lwa4p_extended/meshes/arm_1_link.stl" /-->
           <box size="0.01 0.01 0.01"/>
         </geometry>
@@ -65,5 +64,5 @@
       <calibration rising="${arm_2_ref}"/>
       <dynamics damping="1"/>
-      <limit effort="38" velocity="26.1" lower="-2.0943951" upper="2.0943951"/>
+      <limit effort="48" velocity="1.2566" lower="-2.0943951" upper="2.0943951"/>
       <safety_controller k_position="20" k_velocity="50" soft_lower_limit="${-2.0943 + 0.01}" soft_upper_limit="${2.0943 - 0.01}" />
     </joint>
@@ -95,5 +94,5 @@
       <calibration rising="${arm_3_ref}"/>
       <dynamics damping="1" />
-      <limit effort="38" velocity="26.1" lower="-6.2831853" upper="6.2831853"/>
+      <limit effort="48" velocity="1.2566" lower="-6.2831853" upper="6.2831853"/>
       <safety_controller k_position="20" k_velocity="25" soft_lower_limit="${-6.2831853 + 0.01}" soft_upper_limit="${6.2831853 - 0.01}" />
     </joint>
@@ -130,5 +129,5 @@
       <calibration rising="${arm_4_ref}"/>
       <dynamics damping="1"/>
-      <limit effort="38" velocity="26.1" lower="-2.0943951" upper="2.0943951"/>
+      <limit effort="48" velocity="1.2566" lower="-2.0943951" upper="2.0943951"/>
       <safety_controller k_position="20" k_velocity="25" soft_lower_limit="${-2.0943951 + 0.01}" soft_upper_limit="${2.0943951 - 0.01}" />
     </joint>
@@ -160,5 +159,5 @@
       <calibration rising="${arm_5_ref}"/>
       <dynamics damping="1" />
-      <limit effort="38" velocity="26.1" lower="-6.2831853" upper="6.2831853" />
+      <limit effort="48" velocity="1.2566" lower="-6.2831853" upper="6.2831853" />
       <safety_controller k_position="20" k_velocity="25" soft_lower_limit="${-6.2831853 + 0.01}" soft_upper_limit="${6.2831853 - 0.01}" />
     </joint>
@@ -190,5 +189,5 @@
       <calibration rising="${arm_6_ref}"/>
       <dynamics damping="1" />
-      <limit effort="15" velocity="24.9" lower="-2.0943951" upper="2.0943951" />
+      <limit effort="15" velocity="1.2566" lower="-2.0943951" upper="2.0943951" />
       <safety_controller k_position="20" k_velocity="25" soft_lower_limit="${-2.0943951 + 0.01}" soft_upper_limit="${2.0943951 - 0.01}" />
     </joint>
@@ -220,5 +219,5 @@
       <calibration rising="${arm_7_ref}"/>
       <dynamics damping="1" />
-      <limit effort="15" velocity="24.9" lower="-2.0943951" upper="2.0943951" />
+      <limit effort="15" velocity="1.2566" lower="-2.0943951" upper="2.0943951" />
       <safety_controller k_position="20" k_velocity="25" soft_lower_limit="${-2.0943951 + 0.01}" soft_upper_limit="${2.0943951 - 0.01}" />
     </joint>
