Commit message: tuning urdf, gazebo tags and controlller parameter

File: schunk_lwa4p_extended/urdf/lwa4p_extended.gazebo.xacro (robot description, xacro)
@@ -2,38 +2,102 @@
 <robot xmlns:xacro="http://www.ros.org/wiki/xacro">
   <xacro:macro name="schunk_lwa4p_extended_gazebo" params="name">
+<!--
+	Gazebo tags example for links
+	<gazebo reference="namek">
+      <material value="Schunk/LightGrey"/>
+      <selfCollide>true</selfCollide>
+      <gravity>false</gravity>
+      <dampingFactor>1</dampingFactor>
+      <maxVel>1.0</maxVel>
+      <minDepth>0.0</minDepth>
+      <mu1>1</mu1>
+      <mu2>1</mu2>
+      <fdir1>1 0 0</fdir1>
+      <kp>1000000</kp>
+      <kd>100</kd>
+      <maxContacts>50</maxContacts>
+      <laserRetro>1</laserRetro>
+    </gazebo>
+-->
     <gazebo reference="${name}_base_link">
-      <material value="Schunk/LightGrey" />
-      <turnGravityOff>false</turnGravityOff>
+      <material value="Schunk/LightGrey"/>
       <selfCollide>true</selfCollide>
+      <gravity>false</gravity>
+      <mu1>1</mu1> <!--double, as in reemc_foot-->
+      <mu2>1</mu2> <!--double, as in reemc_foot-->
     </gazebo>
     <gazebo reference="${name}_1_link">
       <material value="Schunk/LightGrey" />
-      <turnGravityOff>false</turnGravityOff>
       <selfCollide>true</selfCollide>
+      <gravity>false</gravity>
+      <mu1>1</mu1> <!--double, as in reemc_foot-->
+      <mu2>1</mu2> <!--double, as in reemc_foot-->
     </gazebo>
     <gazebo reference="${name}_2_link">
-      <turnGravityOff>false</turnGravityOff>
       <selfCollide>true</selfCollide>
+      <gravity>false</gravity>
+      <mu1>1</mu1> <!--double, as in reemc_foot-->
+      <mu2>1</mu2> <!--double, as in reemc_foot-->
     </gazebo>
     <gazebo reference="${name}_3_link">
-      <turnGravityOff>false</turnGravityOff>
       <selfCollide>true</selfCollide>
+      <gravity>false</gravity>
+      <mu1>1</mu1> <!--double, as in reemc_foot-->
+      <mu2>1</mu2> <!--double, as in reemc_foot-->
     </gazebo>
     <gazebo reference="${name}_4_link">
-      <turnGravityOff>false</turnGravityOff>
       <selfCollide>true</selfCollide>
+      <gravity>false</gravity>
+      <mu1>1</mu1> <!--double, as in reemc_foot-->
+      <mu2>1</mu2> <!--double, as in reemc_foot-->
     </gazebo>
     <gazebo reference="${name}_5_link">
-      <turnGravityOff>false</turnGravityOff>
       <selfCollide>true</selfCollide>
+      <gravity>false</gravity>
+      <mu1>1</mu1> <!--double, as in reemc_foot-->
+      <mu2>1</mu2> <!--double, as in reemc_foot-->
     </gazebo>
     <gazebo reference="${name}_6_link">
-      <turnGravityOff>false</turnGravityOff>
       <selfCollide>true</selfCollide>
+      <gravity>false</gravity>
+      <mu1>1</mu1> <!--double, as in reemc_foot-->
+      <mu2>1</mu2> <!--double, as in reemc_foot-->
     </gazebo>
     <gazebo reference="${name}_7_link">
       <material value="Schunk/LightGrey" />
-      <turnGravityOff>false</turnGravityOff>
-      <selfCollide>true</selfCollide>
+      <gravity>false</gravity>
+      <mu1>1</mu1> <!--double, as in reemc_foot-->
+      <mu2>1</mu2> <!--double, as in reemc_foot-->
+    </gazebo>
+<!--
+	Gazebo tags example for joints
+    <gazebo reference="name">
+		<stopCfm>1</stopCfm>
+		<stopErp>1</stopErp>
+		<provideFeedback>1</provideFeedback>
+		<cfmDamping>1</cfmDamping>
+		<fudgeFactor>1</fudgeFactor>
+    </gazebo>
+-->
+    <gazebo reference="${name}_1_joint">
+		<cfmDamping>true</cfmDamping>
+    </gazebo>
+    <gazebo reference="${name}_2_joint">
+		<cfmDamping>true</cfmDamping>
+    </gazebo>
+    <gazebo reference="${name}_3_joint">
+		<cfmDamping>true</cfmDamping>
+    </gazebo>
+    <gazebo reference="${name}_4_joint">
+		<cfmDamping>true</cfmDamping>
+    </gazebo>
+    <gazebo reference="${name}_5_joint">
+		<cfmDamping>true</cfmDamping>
+    </gazebo>
+    <gazebo reference="${name}_6_joint">
+		<cfmDamping>true</cfmDamping>
+    </gazebo>
+    <gazebo reference="${name}_7_joint">
+		<cfmDamping>true</cfmDamping>
     </gazebo>
   </xacro:macro>

File: schunk_lwa4p_extended/urdf/lwa4p_extended.transmission.xacro (robot description, xacro)
@@ -1,61 +1,22 @@
 <?xml version="1.0"?>
 <robot xmlns:xacro="http://www.ros.org/wiki/xacro">
-  <xacro:macro name="schunk_lwa4p_extended_transmission" params="name">
-    <transmission name="${name}_1_trans">
-      <type>transmission_interface/SimpleTransmission</type>
-      <joint name="${name}_1_joint"/>
-      <actuator name="${name}_1_motor">
-        <hardwareInterface>EffortJointInterface</hardwareInterface>
+  <xacro:macro name="schunk_lwa4p_extended_SimpleTransmission" params="jname number">
+	<transmission name="${jname}_${number}_trans">
+	  <type>transmission_interface/SimpleTransmission</type>
+	  <joint name="${jname}_${number}_joint"/>
+      <actuator name="${jname}_${number}_motor">
+		<hardwareInterface>EffortJointInterface</hardwareInterface>
         <mechanicalReduction>1</mechanicalReduction>
       </actuator>
     </transmission>
-    <transmission name="${name}_2_trans">
-      <type>transmission_interface/SimpleTransmission</type>
-      <joint name="${name}_2_joint"/>
-      <actuator name="${name}_2_motor">
-        <hardwareInterface>EffortJointInterface</hardwareInterface>
-        <mechanicalReduction>1</mechanicalReduction>
-      </actuator>
-    </transmission>
-    <transmission name="${name}_3_trans">
-      <type>transmission_interface/SimpleTransmission</type>
-      <joint name="${name}_3_joint"/>
-      <actuator name="${name}_3_motor">
-        <hardwareInterface>EffortJointInterface</hardwareInterface>
-        <mechanicalReduction>1</mechanicalReduction>
-      </actuator>
-    </transmission>
-    <transmission name="${name}_4_trans">
-      <type>transmission_interface/SimpleTransmission</type>
-      <joint name="${name}_4_joint"/>
-      <actuator name="${name}_4_motor">
-        <hardwareInterface>EffortJointInterface</hardwareInterface>
-        <mechanicalReduction>1</mechanicalReduction>
-      </actuator>
-    </transmission>
-    <transmission name="${name}_5_trans">
-      <type>transmission_interface/SimpleTransmission</type>
-      <joint name="${name}_5_joint"/>
-      <actuator name="${name}_5_motor">
-        <hardwareInterface>EffortJointInterface</hardwareInterface>
-        <mechanicalReduction>1</mechanicalReduction>
-      </actuator>
-    </transmission>
-    <transmission name="${name}_6_trans">
-      <type>transmission_interface/SimpleTransmission</type>
-      <joint name="${name}_6_joint"/>
-      <actuator name="${name}_6_motor">
-        <hardwareInterface>EffortJointInterface</hardwareInterface>
-        <mechanicalReduction>1</mechanicalReduction>
-      </actuator>
-    </transmission>
-    <transmission name="${name}_7_trans">
-      <type>transmission_interface/SimpleTransmission</type>
-      <joint name="${name}_7_joint"/>
-      <actuator name="${name}_7_motor">
-        <hardwareInterface>EffortJointInterface</hardwareInterface>
-        <mechanicalReduction>1</mechanicalReduction>
-      </actuator>
-    </transmission>
+   </xacro:macro>
+  <xacro:macro name="schunk_lwa4p_extended_transmission" params="name">
+	<xacro:schunk_lwa4p_extended_SimpleTransmission jname="${name}" number="1"></xacro:schunk_lwa4p_extended_SimpleTransmission>
+	<xacro:schunk_lwa4p_extended_SimpleTransmission jname="${name}" number="2"></xacro:schunk_lwa4p_extended_SimpleTransmission>
+	<xacro:schunk_lwa4p_extended_SimpleTransmission jname="${name}" number="3"></xacro:schunk_lwa4p_extended_SimpleTransmission>
+	<xacro:schunk_lwa4p_extended_SimpleTransmission jname="${name}" number="4"></xacro:schunk_lwa4p_extended_SimpleTransmission>
+	<xacro:schunk_lwa4p_extended_SimpleTransmission jname="${name}" number="5"></xacro:schunk_lwa4p_extended_SimpleTransmission>
+	<xacro:schunk_lwa4p_extended_SimpleTransmission jname="${name}" number="6"></xacro:schunk_lwa4p_extended_SimpleTransmission>
+	<xacro:schunk_lwa4p_extended_SimpleTransmission jname="${name}" number="7"></xacro:schunk_lwa4p_extended_SimpleTransmission>
   </xacro:macro>
 </robot>

File: schunk_lwa4p_extended/urdf/lwa4p_extended.urdf.xacro (robot description, xacro)
@@ -34,10 +34,10 @@
       <axis xyz="0 0 1"/>
       <calibration rising="${arm_1_ref}"/>
-      <dynamics damping="10" />
+      <dynamics damping="1" friction="0"/> <!-- default_damping = 0 [N], default_friction = 0 -->
       <limit effort="370" velocity="2.0" lower="-6.2831853" upper="6.2831853"/>
       <safety_controller k_position="20" k_velocity="50" soft_lower_limit="${-6.2831853 + 0.01}" soft_upper_limit="${6.2831853 - 0.01}" />
     </joint>
     <link name="${name}_1_link">
-      <xacro:box_inertial x="0.01" y="0.01" z="0.01" mass="0.1">
+      <xacro:box_inertial x="0.2" y="0.2" z="0.2" mass="2">
         <origin xyz="0 0 0" rpy="0 0 0" />
       </xacro:box_inertial>
@@ -64,5 +64,5 @@
       <axis xyz="0 0 1"/>
       <calibration rising="${arm_2_ref}"/>
-      <dynamics damping="10" />
+      <dynamics damping="1"/>
       <limit effort="370" velocity="2.0" lower="-2.0943951" upper="2.0943951"/>
       <safety_controller k_position="20" k_velocity="50" soft_lower_limit="${-2.0943 + 0.01}" soft_upper_limit="${2.0943 - 0.01}" />
@@ -94,5 +94,5 @@
       <axis xyz="0 0 1"/>
       <calibration rising="${arm_3_ref}"/>
-      <dynamics damping="5" />
+      <dynamics damping="1" />
       <limit effort="176" velocity="2.0" lower="-6.2831853" upper="6.2831853"/>
       <safety_controller k_position="20" k_velocity="25" soft_lower_limit="${-6.2831853 + 0.01}" soft_upper_limit="${6.2831853 - 0.01}" />
@@ -129,5 +129,5 @@
       <axis xyz="0 0 1" />
       <calibration rising="${arm_4_ref}"/>
-      <dynamics damping="5" />
+      <dynamics damping="1"/>
       <limit effort="176" velocity="2.0" lower="-2.0943951" upper="2.0943951"/>
       <safety_controller k_position="20" k_velocity="25" soft_lower_limit="${-2.0943951 + 0.01}" soft_upper_limit="${2.0943951 - 0.01}" />
@@ -159,5 +159,5 @@
       <axis xyz="0 0 1" />
       <calibration rising="${arm_5_ref}"/>
-      <dynamics damping="5" />
+      <dynamics damping="1" />
       <limit effort="41.6" velocity="2.0" lower="-6.2831853" upper="6.2831853" />
       <safety_controller k_position="20" k_velocity="25" soft_lower_limit="${-6.2831853 + 0.01}" soft_upper_limit="${6.2831853 - 0.01}" />
@@ -189,5 +189,5 @@
       <axis xyz="0 0 1" />
       <calibration rising="${arm_6_ref}"/>
-      <dynamics damping="5" />
+      <dynamics damping="1" />
       <limit effort="20.1" velocity="2.0" lower="-2.0943951" upper="2.0943951" />
       <safety_controller k_position="20" k_velocity="25" soft_lower_limit="${-2.0943951 + 0.01}" soft_upper_limit="${2.0943951 - 0.01}" />
@@ -219,5 +219,5 @@
       <axis xyz="0 0 1" />
       <calibration rising="${arm_7_ref}"/>
-      <dynamics damping="5" />
+      <dynamics damping="1" />
       <limit effort="20.1" velocity="2.0" lower="-2.0943951" upper="2.0943951" />
       <safety_controller k_position="20" k_velocity="25" soft_lower_limit="${-2.0943951 + 0.01}" soft_upper_limit="${2.0943951 - 0.01}" />

Commit message: tabs vs. spaces

File: schunk_lwa4p_extended/urdf/lwa4p_extended.gazebo.xacro (robot description, xacro)
@@ -2,22 +2,22 @@
 <robot xmlns:xacro="http://www.ros.org/wiki/xacro">
   <xacro:macro name="schunk_lwa4p_extended_gazebo" params="name">
-<!--
-	Gazebo tags example for links
-	<gazebo reference="name">
-      <material value="Schunk/LightGrey"/>
-      <selfCollide>true</selfCollide>
-      <gravity>false</gravity>
-      <dampingFactor>1</dampingFactor>
-      <maxVel>1.0</maxVel>
-      <minDepth>0.0</minDepth>
-      <mu1>1</mu1>
-      <mu2>1</mu2>
-      <fdir1>1 0 0</fdir1>
-      <kp>1000000</kp>
-      <kd>100</kd>
-      <maxContacts>50</maxContacts>
-      <laserRetro>1</laserRetro>
-    </gazebo>
--->
+    <!--
+      Gazebo tags example for links
+      <gazebo reference="name">
+        <material value="Schunk/LightGrey"/>
+        <selfCollide>true</selfCollide>
+        <gravity>false</gravity>
+        <dampingFactor>1</dampingFactor>
+        <maxVel>1.0</maxVel>
+        <minDepth>0.0</minDepth>
+        <mu1>1</mu1>
+        <mu2>1</mu2>
+        <fdir1>1 0 0</fdir1>
+        <kp>1000000</kp>
+        <kd>100</kd>
+        <maxContacts>50</maxContacts>
+        <laserRetro>1</laserRetro>
+      </gazebo>
+    -->
     <gazebo reference="${name}_base_link">
       <material value="Schunk/LightGrey"/>
@@ -70,34 +70,34 @@
       <mu2>1</mu2> <!--double, as in reemc_foot-->
     </gazebo>
-<!--
-	Gazebo tags example for joints
+    <!--
+    Gazebo tags example for joints
     <gazebo reference="name">
-		<stopCfm>1</stopCfm>
-		<stopErp>1</stopErp>
-		<provideFeedback>1</provideFeedback>
-		<implicitSpringDamper>1</implicitSpringDamper>
-		<fudgeFactor>1</fudgeFactor>
+      <stopCfm>1</stopCfm>
+      <stopErp>1</stopErp>
+      <provideFeedback>1</provideFeedback>
+      <implicitSpringDamper>1</implicitSpringDamper>
+      <fudgeFactor>1</fudgeFactor>
     </gazebo>
--->
+    -->
     <gazebo reference="${name}_1_joint">
-		<implicitSpringDamper>1</implicitSpringDamper>
+      <implicitSpringDamper>1</implicitSpringDamper>
     </gazebo>
     <gazebo reference="${name}_2_joint">
-		<implicitSpringDamper>1</implicitSpringDamper>
+      <implicitSpringDamper>1</implicitSpringDamper>
     </gazebo>
     <gazebo reference="${name}_3_joint">
-		<implicitSpringDamper>1</implicitSpringDamper>
+      <implicitSpringDamper>1</implicitSpringDamper>
     </gazebo>
     <gazebo reference="${name}_4_joint">
-		<implicitSpringDamper>1</implicitSpringDamper>
+      <implicitSpringDamper>1</implicitSpringDamper>
     </gazebo>
     <gazebo reference="${name}_5_joint">
-		<implicitSpringDamper>1</implicitSpringDamper>
+      <implicitSpringDamper>1</implicitSpringDamper>
     </gazebo>
     <gazebo reference="${name}_6_joint">
-		<implicitSpringDamper>1</implicitSpringDamper>
+      <implicitSpringDamper>1</implicitSpringDamper>
     </gazebo>
     <gazebo reference="${name}_7_joint">
-		<implicitSpringDamper>1</implicitSpringDamper>
+      <implicitSpringDamper>1</implicitSpringDamper>
     </gazebo>
   </xacro:macro>

File: schunk_lwa4p_extended/urdf/lwa4p_extended.transmission.xacro (robot description, xacro)
@@ -2,21 +2,21 @@
 <robot xmlns:xacro="http://www.ros.org/wiki/xacro">
   <xacro:macro name="schunk_lwa4p_extended_SimpleTransmission" params="jname number">
-	<transmission name="${jname}_${number}_trans">
-	  <type>transmission_interface/SimpleTransmission</type>
-	  <joint name="${jname}_${number}_joint"/>
+    <transmission name="${jname}_${number}_trans">
+      <type>transmission_interface/SimpleTransmission</type>
+      <joint name="${jname}_${number}_joint"/>
       <actuator name="${jname}_${number}_motor">
-		<hardwareInterface>EffortJointInterface</hardwareInterface>
+        <hardwareInterface>EffortJointInterface</hardwareInterface>
         <mechanicalReduction>1</mechanicalReduction>
       </actuator>
     </transmission>
-   </xacro:macro>
+  </xacro:macro>
   <xacro:macro name="schunk_lwa4p_extended_transmission" params="name">
-	<xacro:schunk_lwa4p_extended_SimpleTransmission jname="${name}" number="1"></xacro:schunk_lwa4p_extended_SimpleTransmission>
-	<xacro:schunk_lwa4p_extended_SimpleTransmission jname="${name}" number="2"></xacro:schunk_lwa4p_extended_SimpleTransmission>
-	<xacro:schunk_lwa4p_extended_SimpleTransmission jname="${name}" number="3"></xacro:schunk_lwa4p_extended_SimpleTransmission>
-	<xacro:schunk_lwa4p_extended_SimpleTransmission jname="${name}" number="4"></xacro:schunk_lwa4p_extended_SimpleTransmission>
-	<xacro:schunk_lwa4p_extended_SimpleTransmission jname="${name}" number="5"></xacro:schunk_lwa4p_extended_SimpleTransmission>
-	<xacro:schunk_lwa4p_extended_SimpleTransmission jname="${name}" number="6"></xacro:schunk_lwa4p_extended_SimpleTransmission>
-	<xacro:schunk_lwa4p_extended_SimpleTransmission jname="${name}" number="7"></xacro:schunk_lwa4p_extended_SimpleTransmission>
+    <xacro:schunk_lwa4p_extended_SimpleTransmission jname="${name}" number="1"></xacro:schunk_lwa4p_extended_SimpleTransmission>
+    <xacro:schunk_lwa4p_extended_SimpleTransmission jname="${name}" number="2"></xacro:schunk_lwa4p_extended_SimpleTransmission>
+    <xacro:schunk_lwa4p_extended_SimpleTransmission jname="${name}" number="3"></xacro:schunk_lwa4p_extended_SimpleTransmission>
+    <xacro:schunk_lwa4p_extended_SimpleTransmission jname="${name}" number="4"></xacro:schunk_lwa4p_extended_SimpleTransmission>
+    <xacro:schunk_lwa4p_extended_SimpleTransmission jname="${name}" number="5"></xacro:schunk_lwa4p_extended_SimpleTransmission>
+    <xacro:schunk_lwa4p_extended_SimpleTransmission jname="${name}" number="6"></xacro:schunk_lwa4p_extended_SimpleTransmission>
+    <xacro:schunk_lwa4p_extended_SimpleTransmission jname="${name}" number="7"></xacro:schunk_lwa4p_extended_SimpleTransmission>
   </xacro:macro>
 </robot>
