Commit message: playing with the physics properties

File: schunk_lwa4p_extended/urdf/lwa4p_extended.gazebo.xacro (robot description, xacro)
@@ -23,50 +23,50 @@
       <material value="Schunk/LightGrey"/>
       <selfCollide>true</selfCollide>
-      <gravity>false</gravity>
-      <mu1>1</mu1> <!--double, as in reemc_foot-->
-      <mu2>1</mu2> <!--double, as in reemc_foot-->
+      <!--gravity>false</gravity-->
+      <mu1>0.5</mu1> <!--double, as in reemc_foot-->
+      <mu2>0.5</mu2> <!--double, as in reemc_foot-->
     </gazebo>
     <gazebo reference="${name}_1_link">
       <material value="Schunk/LightGrey" />
       <selfCollide>true</selfCollide>
-      <gravity>false</gravity>
-      <mu1>1</mu1> <!--double, as in reemc_foot-->
-      <mu2>1</mu2> <!--double, as in reemc_foot-->
+      <!--gravity>false</gravity-->
+      <mu1>0.5</mu1> <!--double, as in reemc_foot-->
+      <mu2>0.5</mu2> <!--double, as in reemc_foot-->
     </gazebo>
     <gazebo reference="${name}_2_link">
       <selfCollide>true</selfCollide>
-      <gravity>false</gravity>
-      <mu1>1</mu1> <!--double, as in reemc_foot-->
-      <mu2>1</mu2> <!--double, as in reemc_foot-->
+      <!--gravity>false</gravity-->
+      <mu1>0.5</mu1> <!--double, as in reemc_foot-->
+      <mu2>0.5</mu2> <!--double, as in reemc_foot-->
     </gazebo>
     <gazebo reference="${name}_3_link">
       <selfCollide>true</selfCollide>
-      <gravity>false</gravity>
-      <mu1>1</mu1> <!--double, as in reemc_foot-->
-      <mu2>1</mu2> <!--double, as in reemc_foot-->
+      <!--gravity>false</gravity-->
+      <mu1>0.5</mu1> <!--double, as in reemc_foot-->
+      <mu2>0.5</mu2> <!--double, as in reemc_foot-->
     </gazebo>
     <gazebo reference="${name}_4_link">
       <selfCollide>true</selfCollide>
-      <gravity>false</gravity>
-      <mu1>1</mu1> <!--double, as in reemc_foot-->
-      <mu2>1</mu2> <!--double, as in reemc_foot-->
+      <!--gravity>false</gravity-->
+      <mu1>0.5</mu1> <!--double, as in reemc_foot-->
+      <mu2>0.5</mu2> <!--double, as in reemc_foot-->
     </gazebo>
     <gazebo reference="${name}_5_link">
       <selfCollide>true</selfCollide>
-      <gravity>false</gravity>
-      <mu1>1</mu1> <!--double, as in reemc_foot-->
-      <mu2>1</mu2> <!--double, as in reemc_foot-->
+      <!--gravity>false</gravity-->
+      <mu1>0.5</mu1> <!--double, as in reemc_foot-->
+      <mu2>0.5</mu2> <!--double, as in reemc_foot-->
     </gazebo>
     <gazebo reference="${name}_6_link">
       <selfCollide>true</selfCollide>
-      <gravity>false</gravity>
-      <mu1>1</mu1> <!--double, as in reemc_foot-->
-      <mu2>1</mu2> <!--double, as in reemc_foot-->
+      <!--gravity>false</gravity-->
+      <mu1>0.5</mu1> <!--double, as in reemc_foot-->
+      <mu2>0.5</mu2> <!--double, as in reemc_foot-->
     </gazebo>
     <gazebo reference="${name}_7_link">
       <material value="Schunk/LightGrey" />
-      <gravity>false</gravity>
-      <mu1>1</mu1> <!--double, as in reemc_foot-->
-      <mu2>1</mu2> <!--double, as in reemc_foot-->
+      <!--gravity>false</gravity-->
+      <mu1>0.5</mu1> <!--double, as in reemc_foot-->
+      <mu2>0.5</mu2> <!--double, as in reemc_foot-->
     </gazebo>
     <!--
@@ -81,23 +81,23 @@
     -->
     <gazebo reference="${name}_1_joint">
-      <implicitSpringDamper>1</implicitSpringDamper>
+      <implicitSpringDamper>true</implicitSpringDamper>
     </gazebo>
     <gazebo reference="${name}_2_joint">
-      <implicitSpringDamper>1</implicitSpringDamper>
+      <implicitSpringDamper>true</implicitSpringDamper>
     </gazebo>
     <gazebo reference="${name}_3_joint">
-      <implicitSpringDamper>1</implicitSpringDamper>
+      <implicitSpringDamper>true</implicitSpringDamper>
     </gazebo>
     <gazebo reference="${name}_4_joint">
-      <implicitSpringDamper>1</implicitSpringDamper>
+      <implicitSpringDamper>true</implicitSpringDamper>
     </gazebo>
     <gazebo reference="${name}_5_joint">
-      <implicitSpringDamper>1</implicitSpringDamper>
+      <implicitSpringDamper>true</implicitSpringDamper>
     </gazebo>
     <gazebo reference="${name}_6_joint">
-      <implicitSpringDamper>1</implicitSpringDamper>
+      <implicitSpringDamper>true</implicitSpringDamper>
     </gazebo>
     <gazebo reference="${name}_7_joint">
-      <implicitSpringDamper>1</implicitSpringDamper>
+      <implicitSpringDamper>true</implicitSpringDamper>
     </gazebo>
   </xacro:macro>

File: schunk_lwa4p_extended/urdf/lwa4p_extended.urdf.xacro (robot description, xacro)
@@ -34,12 +34,14 @@
       <axis xyz="0 0 1"/>
       <calibration rising="${arm_1_ref}"/>
-      <dynamics damping="1" friction="0"/> <!-- default_damping = 0 [N], default_friction = 0 -->
+      <dynamics damping="0.7" friction="0"/> <!-- default_damping = 0 [N], default_friction = 0 -->
       <limit effort="81.5" velocity="0.42" lower="-6.2831853" upper="6.2831853"/>
       <safety_controller k_position="20" k_velocity="50" soft_lower_limit="${-6.2831853 + 0.01}" soft_upper_limit="${6.2831853 - 0.01}" />
     </joint>
     <link name="${name}_1_link">
-      <xacro:box_inertial x="0.2" y="0.2" z="0.2" mass="2">
-        <origin xyz="0 0 0" rpy="0 0 0" />
-      </xacro:box_inertial>
+      <inertial>
+        <origin xyz="0.0 0.0 0.0" rpy="0 0 0"/>
+        <mass value="1.0"/>
+        <inertia ixx="0.01" ixy="0.0" ixz="0.0" iyy="0.01" iyz="0.0" izz="0.01" />
+      </inertial>
       <visual>
         <origin xyz="0 0 0" rpy="0 0 0" />
@@ -63,5 +65,5 @@
       <axis xyz="0 0 1"/>
       <calibration rising="${arm_2_ref}"/>
-      <dynamics damping="1"/>
+      <dynamics damping="0.7" friction="0"/> <!-- default_damping = 0 [N], default_friction = 0 -->
       <limit effort="48" velocity="1.2566" lower="-2.0943951" upper="2.0943951"/>
       <safety_controller k_position="20" k_velocity="50" soft_lower_limit="${-2.0943 + 0.01}" soft_upper_limit="${2.0943 - 0.01}" />
@@ -93,5 +95,5 @@
       <axis xyz="0 0 1"/>
       <calibration rising="${arm_3_ref}"/>
-      <dynamics damping="1" />
+      <dynamics damping="0.7" friction="0"/> <!-- default_damping = 0 [N], default_friction = 0 -->
       <limit effort="48" velocity="1.2566" lower="-6.2831853" upper="6.2831853"/>
       <safety_controller k_position="20" k_velocity="25" soft_lower_limit="${-6.2831853 + 0.01}" soft_upper_limit="${6.2831853 - 0.01}" />
@@ -128,5 +130,5 @@
       <axis xyz="0 0 1" />
       <calibration rising="${arm_4_ref}"/>
-      <dynamics damping="1"/>
+      <dynamics damping="0.7" friction="0"/> <!-- default_damping = 0 [N], default_friction = 0 -->
       <limit effort="48" velocity="1.2566" lower="-2.0943951" upper="2.0943951"/>
       <safety_controller k_position="20" k_velocity="25" soft_lower_limit="${-2.0943951 + 0.01}" soft_upper_limit="${2.0943951 - 0.01}" />
@@ -158,5 +160,5 @@
       <axis xyz="0 0 1" />
       <calibration rising="${arm_5_ref}"/>
-      <dynamics damping="1" />
+      <dynamics damping="0.7" friction="0"/> <!-- default_damping = 0 [N], default_friction = 0 -->
       <limit effort="48" velocity="1.2566" lower="-6.2831853" upper="6.2831853" />
       <safety_controller k_position="20" k_velocity="25" soft_lower_limit="${-6.2831853 + 0.01}" soft_upper_limit="${6.2831853 - 0.01}" />
@@ -188,5 +190,5 @@
       <axis xyz="0 0 1" />
       <calibration rising="${arm_6_ref}"/>
-      <dynamics damping="1" />
+      <dynamics damping="0.7" friction="0"/> <!-- default_damping = 0 [N], default_friction = 0 -->
       <limit effort="15" velocity="1.2566" lower="-2.0943951" upper="2.0943951" />
       <safety_controller k_position="20" k_velocity="25" soft_lower_limit="${-2.0943951 + 0.01}" soft_upper_limit="${2.0943951 - 0.01}" />
@@ -218,5 +220,5 @@
       <axis xyz="0 0 1" />
       <calibration rising="${arm_7_ref}"/>
-      <dynamics damping="1" />
+      <dynamics damping="0.7" friction="0"/> <!-- default_damping = 0 [N], default_friction = 0 -->
       <limit effort="15" velocity="1.2566" lower="-2.0943951" upper="2.0943951" />
       <safety_controller k_position="20" k_velocity="25" soft_lower_limit="${-2.0943951 + 0.01}" soft_upper_limit="${2.0943951 - 0.01}" />
