Commit message: give podest more space - stops bouncing

File: schunk_lwa4d/urdf/robot.urdf.xacro (robot description, xacro)
@@ -20,5 +20,5 @@
             arm_6_ref="${arm_6_ref}"
             arm_7_ref="${arm_7_ref}">
-    <origin xyz="0 0 0.01" rpy="0 0 0" /> <!--slightly above gazebo plane-->
+    <origin xyz="0 0 0.026" rpy="0 0 0" /> <!--slightly above gazebo plane-->
   </xacro:schunk_lwa4d>
   <!-- gazebo_plugin for arm -->

File: schunk_lwa4p/urdf/robot.urdf.xacro (robot description, xacro)
@@ -19,5 +19,5 @@
             arm_5_ref="${arm_5_ref}"
             arm_6_ref="${arm_6_ref}">
-    <origin xyz="0 0 0.01" rpy="0 0 0" /> <!--slightly above gazebo plane-->
+    <origin xyz="0 0 0.052" rpy="0 0 0" /> <!--slightly above gazebo plane-->
   </xacro:schunk_lwa4p>
   <!-- gazebo_plugin for arm -->

File: schunk_lwa4p_extended/urdf/robot.urdf.xacro (robot description, xacro)
@@ -20,5 +20,5 @@
             arm_6_ref="${arm_6_ref}"
             arm_7_ref="${arm_7_ref}">
-    <origin xyz="0 0 0.01" rpy="0 0 0" /> <!--slightly above gazebo plane-->
+    <origin xyz="0 0 0.026" rpy="0 0 0" /> <!--slightly above gazebo plane-->
   </xacro:schunk_lwa4p_extended>
   <!-- gazebo_plugin for arm -->
